File: HE60/HE60.kicad_pcb (KiCad board)
At the start: 2 copper layers, 284.7 x 94.2 mm, 331 parts, among them J1 TYPE-C-31-M-12, J2 JST_SH, SW1 TS-1187A-B-A-B, SW2 TS-1187A-B-A-B, U1 USBLC6-2SC6, U2 TLV75733PDBV, U3 XC6206P332MR-G, U4 AT32F405RCT7, Y1 X322512MSB4SI

Commit message: layout: add arrows and top 3 block
Parts:
- removed PCB1: H60, HE60:H60
- added AM10: SN74LV4051A, Package_SO:TSSOP-16_4.4x5mm_P0.65mm, B.Cu at (351.8, 186.4)
- added C161: 100n, Capacitor_SMD:C_0402_1005Metric, B.Cu at (450.6, 154.7)
- added C170: 100n, Capacitor_SMD:C_0402_1005Metric, B.Cu at (469.2, 154.8)
- added C171: 4.7n, Capacitor_SMD:C_0402_1005Metric, B.Cu at (474.9, 154.8)
- added C172: 100n, Capacitor_SMD:C_0402_1005Metric, B.Cu at (469.4, 231.0)
- added C173: 4.7n, Capacitor_SMD:C_0402_1005Metric, B.Cu at (456.4, 154.9)
- added C174: 100n, Capacitor_SMD:C_0402_1005Metric, B.Cu at (451.1, 211.9)
- added C175: 4.7n, Capacitor_SMD:C_0402_1005Metric, B.Cu at (437.1, 154.9)
- added C178: 100n, Capacitor_SMD:C_0402_1005Metric, B.Cu at (450.9, 232.4)
- added C179: 4.7n, Capacitor_SMD:C_0402_1005Metric, B.Cu at (475.2, 231.0)
- added C180: 100n, Capacitor_SMD:C_0402_1005Metric, B.Cu at (431.8, 231.3)
- added C181: 4.7n, Capacitor_SMD:C_0402_1005Metric, B.Cu at (436.8, 231.2)
- added C182: 100n, Capacitor_SMD:C_0402_1005Metric, B.Cu at (431.6, 155.2)
- added C183: 4.7n, Capacitor_SMD:C_0402_1005Metric, B.Cu at (455.9, 230.8)
- added C184: 100n, Capacitor_SMD:C_0402_1005Metric, B.Cu at (347.4, 183.4)
- added C185: 4.7n, Capacitor_SMD:C_0402_1005Metric, B.Cu at (456.4, 211.7)
- added HE74: MT9102ET, Package_TO_SOT_SMD:SOT-23-3, B.Cu at (472.5, 156.8)
- added HE75: MT9102ET, Package_TO_SOT_SMD:SOT-23-3, B.Cu at (453.4, 156.8)
- added HE76: MT9102ET, Package_TO_SOT_SMD:SOT-23-3, B.Cu at (434.4, 156.8)
- added HE78: MT9102ET, Package_TO_SOT_SMD:SOT-23-3, B.Cu at (472.5, 233.1)
- added HE79: MT9102ET, Package_TO_SOT_SMD:SOT-23-3, B.Cu at (434.4, 233.1)
- added HE80: MT9102ET, Package_TO_SOT_SMD:SOT-23-3, B.Cu at (453.4, 233.1)
- added HE81: MT9102ET, Package_TO_SOT_SMD:SOT-23-3, B.Cu at (453.4, 214.0)
- added J3: JST_SH, Connector_JST:JST_SH_SM04B-SRSS-TB_1x04-1MP_P1.00mm_Horizontal, B.Cu at (416.7, 196.0)
- added J5: JST_SH, Connector_JST:JST_SH_SM04B-SRSS-TB_1x04-1MP_P1.00mm_Horizontal, F.Cu at (416.7, 190.4)
- moved AM1 200.2 mm to (239.2, 166.4)
- moved AM2 200.2 mm to (296.3, 166.4)
- moved AM3 200.2 mm to (224.9, 185.4)
- moved AM4 200.2 mm to (301.1, 185.4)
- moved AM5 200.2 mm to (215.3, 204.5)
- moved AM6 200.2 mm to (305.8, 204.5)
- moved AM7 200.2 mm to (205.8, 223.6)
- moved AM8 200.2 mm to (253.4, 223.6)
- moved AM9 200.2 mm to (301.1, 223.6)
- moved C1 200.2 mm to (146.5, 157.7)
- moved C10 200.2 mm to (222.7, 156.1)
- moved C100 200.2 mm to (284.6, 213.2)
- moved C101 200.2 mm to (298.5, 213.2)
- moved C102 200.2 mm to (303.7, 213.2)
- moved C103 200.2 mm to (317.5, 213.2)
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Connections:
- U4 pad 16: unconnected-(U4-PA2-Pad16) -> MUX_OUT_10
- U4 pad 42: unconnected-(U4-PA9-Pad42) -> UART_TX
- U4 pad 43: unconnected-(U4-PA10-Pad43) -> UART_RX
- U4 pad 46: unconnected-(U4-PA13-Pad46) -> SWDIO
- U4 pad 49: unconnected-(U4-PA14-Pad49) -> SWCLK
Routing:
- net UART_TX: track 0.00 -> 291.7 mm, vias 0 -> 3
- net UART_RX: track 0.00 -> 283.3 mm, vias 0 -> 3
- net MUX_OUT_10: track 0.00 -> 209.6 mm, vias 0 -> 2
- net +3.3VA: track 1712.8 -> 1914.4 mm, vias 19 -> 33
- net HE74: track 0.00 -> 164.9 mm
- net HE76: track 0.00 -> 160.9 mm
- net HE70: track 0.00 -> 154.3 mm
- net HE77: track 0.00 -> 146.1 mm
- net HE71: track 0.00 -> 135.1 mm
- net HE75: track 0.00 -> 125.6 mm
- net HE72: track 0.00 -> 114.4 mm
- net MUX_SELECT_0: track 342.4 -> 392.6 mm, vias 10 -> 12
- net MUX_SELECT_1: track 341.8 -> 390.3 mm
- net MUX_SELECT_2: track 343.0 -> 390.6 mm, vias 10 -> 12
- net GND: track 228.4 -> 238.2 mm, vias 2024 -> 2031
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Other:
- board size 284.7 x 94.2 mm -> 347.6 x 97.2 mm
- board text added: "TODO: - Cutout for module JST - Mounting holes for PCB and Plate connecting"
