File: HE60/HE60.kicad_pcb (KiCad board)
At the start: 2 copper layers, 284.7 x 94.2 mm, 331 parts, among them J1 TYPE-C-31-M-12, J2 JST_SH, SW1 TS-1187A-B-A-B, SW2 TS-1187A-B-A-B, U1 USBLC6-2SC6, U2 TLV75733PDBV, U3 XC6206P332MR-G, U4 AT32F405RCT7, Y1 X322512MSB4SI

Commit message: del footprints in wkl area
Parts:
- removed C117, C135: 100n, Capacitor_SMD:C_0402_1005Metric
- removed C118, C136: 4.7n, Capacitor_SMD:C_0402_1005Metric
- removed HE59, HE68: MT9102ET, Package_TO_SOT_SMD:SOT-23-3
- removed MX60, MX74: 1.25U, HE60:MX-1.25U
- removed MX61, MX73: 1U, HE60:MX-1U
Routing:
- net HE68: track 89.5 -> 80.3 mm
- net +3.3VA: track 1712.8 -> 1706.5 mm
- net GND: track 228.4 -> 223.4 mm, vias 2024 -> 2018
- net HE59: track 43.3 -> 41.5 mm

Commit message: flip stabilizer mounting holes to clear wkl blockers
Parts:
- turned MX43 to 180 degrees
- turned MX44 to 180 degrees
- turned MX56 to 180 degrees

Commit message: add models for 1u
https://grabcad.com/library/cherry-mx-switches-mx-1
Parts:
- added AM10: SN74LV4051A, Package_SO:TSSOP-16_4.4x5mm_P0.65mm, B.Cu at (77.3, 19.9)
- added C117: 100n, Capacitor_SMD:C_0402_1005Metric, F.Cu at (149.5, -31.1)
- added C118: 4.7n, Capacitor_SMD:C_0402_1005Metric, F.Cu at (148.7, -25.3)
- added C135: 100n, Capacitor_SMD:C_0402_1005Metric, F.Cu at (148.7, -23.3)
- added C136: 4.7n, Capacitor_SMD:C_0402_1005Metric, F.Cu at (148.7, -21.3)
- added C161: 100n, Capacitor_SMD:C_0402_1005Metric, F.Cu at (74.1, -22.0)
- added HE59: MT9102ET, Package_TO_SOT_SMD:SOT-23-3, F.Cu at (146.9, -38.5)
- added HE68: MT9102ET, Package_TO_SOT_SMD:SOT-23-3, F.Cu at (163.2, -32.2)
- added J3: Conn_01x09_MountingPin, Connector_JST:JST_SH_SM09B-SRSS-TB_1x09-1MP_P1.00mm_Horizontal, B.Cu at (68.0, 17.9)
- added J4: Conn_01x06_MountingPin, Connector_JST:JST_SH_SM06B-SRSS-TB_1x06-1MP_P1.00mm_Horizontal, B.Cu at (47.1, 19.5)
- J2: value JST_SH -> SWD; footprint Connector_JST:JST_SH_SM04B-SRSS-TB_1x04-1MP_P1.00mm_Horizontal -> Connector_PinHeader_2.54mm:PinHeader_1x04_P2.54mm_Vertical; moved to F.Cu
- moved J2 70.6 mm to (84.3, -41.5), turned to 0 degrees
Connections:
- J2 pad 1: VBUS -> +3.3V
- J2 pad 2: USB_PLUG_D- -> SWDIO
- J2 pad 3: USB_PLUG_D+ -> SWCLK
- U4 pad 16: unconnected-(U4-PA2-Pad16) -> MUX_OUT_10
- U4 pad 42: unconnected-(U4-PA9-Pad42) -> AT32_TX
- U4 pad 43: unconnected-(U4-PA10-Pad43) -> AT32_RX
- U4 pad 46: unconnected-(U4-PA13-Pad46) -> SWDIO
- U4 pad 49: unconnected-(U4-PA14-Pad49) -> SWCLK
Routing:
- net MUX_OUT_10: track 0.00 -> 65.9 mm, vias 0 -> 4
- net HE74: track 0.00 -> 12.5 mm
- net HE76: track 0.00 -> 11.7 mm
- net HE75: track 0.00 -> 11.4 mm
- net HE2: track 80.4 -> 86.8 mm, vias 0 -> 2
- net HE3: track 62.1 -> 67.7 mm, vias 0 -> 2
- net HE70: track 0.00 -> 4.73 mm
- net HE73: track 0.00 -> 4.63 mm
- net HE71: track 0.00 -> 4.59 mm
- net HE72: track 0.00 -> 4.48 mm
- net HE4: track 43.7 -> 46.7 mm, vias 0 -> 2
- net MUX_SELECT_0: track 342.4 -> 344.1 mm
- net MUX_SELECT_1: track 341.8 -> 343.4 mm
- net MUX_SELECT_2: track 343.0 -> 344.4 mm
- net GND: track 223.4 -> 224.1 mm, vias 2018 -> 2009
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Other:
- board text added: "TODO"
- board text added: "TODO THESE"
- board text added: "TODO: VA to bottom bus"
