File: HE60/HE60.kicad_pcb (KiCad board)
At the start: 2 copper layers, 284.7 x 94.2 mm, 331 parts, among them J1 TYPE-C-31-M-12, J2 SWD, J3 Conn_01x09_MountingPin, J4 Conn_01x06_MountingPin, SW1 TS-1187A-B-A-B, SW2 TS-1187A-B-A-B, U1 USBLC6-2SC6, U2 TLV75733PDBV, U3 XC6206P332MR-G, U4 AT32F405RCT7, Y1 X322512MSB4SI

Commit message: add keycaps to 3d model
Parts:
- moved C117 156.1 mm to (10.3, 39.6)
- moved C118 156.1 mm to (9.53, 45.5)
- moved C135 156.1 mm to (9.53, 47.4)
- moved C136 156.1 mm to (9.53, 49.4)
- moved HE59 156.1 mm to (7.75, 32.3)
- moved HE68 156.1 mm to (24.0, 38.5)
- moved J2 105.6 mm to (2.62, 25.3)
- moved C161 95.5 mm to (2.81, 41.5)
Changed lines of the file:
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@@
 			)
 		)
+		(model "${KIPRJMOD}/3d_mondels/keycaps-shoppster/k7u.step"
+			(offset
+				(xyz -455.7 -52.35 11.5)
+			)
+			(scale
+				(xyz 1 1 1)
+			)
+			(rotate
+				(xyz -0 -0 -0)
+			)
+		)
 	)
 	(footprint "HE60:ToolingHole"
@@
 			)
 		)
+		(model "${KIPRJMOD}/3d_mondels/keycaps-shoppster/k2.25u.step"
+			(offset
+				(xyz -303 -248.1 11.5)
+			)
+			(scale
+				(xyz 1 1 1)
+			)
+			(rotate
+				(xyz -0 -0 -0)
+			)
+		)
 	)
 	(footprint "HE60:MX-1U"
@@
 			)
 		)
+		(model "${KIPRJMOD}/3d_mondels/keycaps-shoppster/k1.75.step"
+			(offset
+				(xyz -190.75 -248 11.5)
+			)
+			(scale
+				(xyz 1 1 1)
+			)
+			(rotate
+				(xyz -0 -0 -0)
+			)
+		)
 	)
 	(footprint "Capacitor_SMD:C_0402_1005Metric"
 		(layer "F.Cu")
-		(at 149.505 -31.075)
+		(at 10.33 39.65)
 		(descr "Capacitor SMD 0402 (1005 Metric), square (rectangular) end terminal, IPC-7351 nominal, (Body size source: IPC-SM-782 page 76, https://www.pcb-3d.com/wordpress/wp-content/uploads/ipc-sm-782a_amendment_1_and_2.pdf), generated with kicad-footprint-generator")
 		(tags "capacitor")
@@
 	(footprint "Capacitor_SMD:C_0402_1005Metric"
 		(layer "F.Cu")
-		(at 148.705 -21.325)
+		(at 9.53 49.4)
 		(descr "Capacitor SMD 0402 (1005 Metric), square (rectangular) end terminal, IPC-7351 nominal, (Body size source: IPC-SM-782 page 76, https://www.pcb-3d.com/wordpress/wp-content/uploads/ipc-sm-782a_amendment_1_and_2.pdf), generated with kicad-footprint-generator")
 		(tags "capacitor")
@@
 			)
 		)
+		(model "${KIPRJMOD}/3d_mondels/keycaps-shoppster/k1.5.step"
+			(offset
+				(xyz -141.75 -248.13 11.5)
+			)
+			(scale
+				(xyz 1 1 1)
+			)
+			(rotate
+				(xyz -0 -0 -0)
+			)
+		)
 	)
 	(footprint "HE60:MX-1U"
@@
 			)
 		)
+		(model "${KIPRJMOD}/3d_mondels/keycaps-shoppster/k2.25u.step"
+			(offset
+				(xyz -303 -248.1 11.5)
+			)
+			(scale
+				(xyz 1 1 1)
+			)
+			(rotate
+				(xyz -0 -0 -0)
+			)
+		)
 	)
 	(footprint "HE60:MX-1U"
@@
 			)
 		)
+		(model "${KIPRJMOD}/3d_mondels/keycaps-shoppster/k1.5.step"
+			(offset
+				(xyz -141.75 -248.13 11.5)
+			)
+			(scale
+				(xyz 1 1 1)
+			)
+			(rotate
+				(xyz -0 -0 -0)
+			)
+		)
 	)
 	(footprint "HE60:MX-1.5U"
@@
 			)
 		)
+		(model "${KIPRJMOD}/3d_mondels/keycaps-shoppster/k1.5.step"
+			(offset
+				(xyz -141.75 -248.13 11.5)
+			)
+			(scale
+				(xyz 1 1 1)
+			)
+			(rotate
+				(xyz -0 -0 -0)
+			)
+		)
 	)
 	(footprint "HE60:MX-1U"
@@
 	(footprint "Capacitor_SMD:C_0402_1005Metric"
 		(layer "F.Cu")
-		(at 148.705 -23.295)
+		(at 9.53 47.43)
 		(descr "Capacitor SMD 0402 (1005 Metric), square (rectangular) end terminal, IPC-7351 nominal, (Body size source: IPC-SM-782 page 76, https://www.pcb-3d.com/wordpress/wp-content/uploads/ipc-sm-782a_amendment_1_and_2.pdf), generated with kicad-footprint-generator")
 		(tags "capacitor")
@@
 			)
 		)
+		(model "${KIPRJMOD}/3d_mondels/keycaps-shoppster/k1.5.step"
+			(offset
+				(xyz -141.75 -248.13 11.5)
+			)
+			(scale
+				(xyz 1 1 1)
+			)
+			(rotate
+				(xyz -0 -0 -0)
+			)
+		)
 	)
 	(footprint "HE60:H60"
@@
 	(footprint "Connector_PinHeader_2.54mm:PinHeader_1x04_P2.54mm_Vertical"
 		(layer "F.Cu")
-		(at 84.3475 -41.505)
+		(at 2.625 25.325)
 		(descr "Through hole straight pin header, 1x04, 2.54mm pitch, single row")
 		(tags "Through hole pin header THT 1x04 2.54mm single row")
@@
 			)
 		)
+		(model "${KIPRJMOD}/3d_mondels/keycaps-shoppster/k1.75.step"
+			(offset
+				(xyz -190.75 -248 11.5)
+			)
+			(scale
+				(xyz 1 1 1)
+			)
+			(rotate
+				(xyz -0 -0 -0)
+			)
+		)
 	)
 	(footprint "HE60:MX-1U"
@@
 	(footprint "Package_TO_SOT_SMD:SOT-23-3"
 		(layer "F.Cu")
-		(at 163.2 -32.1875)
+		(at 24.025 38.5375)
 		(descr "SOT, 3 Pin (JEDEC MO-178 inferred 3-pin variant https://www.jedec.org/document_search?search_api_views_fulltext=MO-178), generated with kicad-footprint-generator ipc_gullwing_generator.py")
 		(tags "SOT TO_SOT_SMD")
@@
 			)
 		)
+		(model "${KIPRJMOD}/3d_mondels/keycaps-shoppster/k1.5.step"
+			(offset
+				(xyz -141.75 -248.13 11.5)
+			)
+			(scale
+				(xyz 1 1 1)
+			)
+			(rotate
+				(xyz -0 -0 -0)
+			)
+		)
 	)
 	(footprint "HE60:MX-1.25U"
@@
 		(embedded_fonts no)
 		(model "${KIPRJMOD}/3d_mondels/cherry-mx-switches-mx-1.snapshot.16/MX .STEP"
+			(hide yes)
 			(offset
 				(xyz -7.35 -7.35 5.95)
@@
 	(footprint "Package_TO_SOT_SMD:SOT-23-3"
 		(layer "F.Cu")
-		(at 146.925 -38.4625)
+		(at 7.75 32.2625)
 		(descr "SOT, 3 Pin (JEDEC MO-178 inferred 3-pin variant https://www.jedec.org/document_search?search_api_views_fulltext=MO-178), generated with kicad-footprint-generator ipc_gullwing_generator.py")
 		(tags "SOT TO_SOT_SMD")
@@
 			)
 		)
+		(model "${KIPRJMOD}/3d_mondels/keycaps-shoppster/k1.5.step"
+			(offset
+				(xyz -141.75 -248.13 11.5)
+			)
+			(scale
+				(xyz 1 1 1)
+			)
+			(rotate
+				(xyz -0 -0 -0)
+			)
+		)
 	)
 	(footprint "Capacitor_SMD:C_0402_1005Metric"
 		(layer "F.Cu")
-		(at 148.705 -25.265)
+		(at 9.53 45.46)
 		(descr "Capacitor SMD 0402 (1005 Metric), square (rectangular) end terminal, IPC-7351 nominal, (Body size source: IPC-SM-782 page 76, https://www.pcb-3d.com/wordpress/wp-content/uploads/ipc-sm-782a_amendment_1_and_2.pdf), generated with kicad-footprint-generator")
 		(tags "capacitor")
@@
 	(footprint "Capacitor_SMD:C_0402_1005Metric"
 		(layer "F.Cu")
-		(at 74.1 -21.975)
+		(at 2.805 41.5)
 		(descr "Capacitor SMD 0402 (1005 Metric), square (rectangular) end terminal, IPC-7351 nominal, (Body size source: IPC-SM-782 page 76, https://www.pcb-3d.com/wordpress/wp-content/uploads/ipc-sm-782a_amendment_1_and_2.pdf), generated with kicad-footprint-generator")
 		(tags "capacitor")
