File: HE60/HE60.kicad_sch (KiCad schematic)
At the start: 331 parts, among them J1 TYPE-C-31-M-12, J2 JST_SH, SW1 TS-1187A-B-A-B, SW2 TS-1187A-B-A-B, U1 USBLC6-2SC6, U2 TLV75733PDBV, U3 XC6206P332MR-G, U4 AT32F405RCT7, Y1 X322512MSB4SI

Commit message: sch: add another adc mux and 8 more HE sensors
Parts:
- added AM10: SN74LV4051A, Package_SO:TSSOP-16_4.4x5mm_P0.65mm, symbol 4xxx:4051
- added C161, C170, C172, C174, C176, C178, C180, C182, C184: 100n, Capacitor_SMD:C_0402_1005Metric, symbol Device:C
- added C171, C173, C175, C177, C179, C181, C183, C185: 4.7n, Capacitor_SMD:C_0402_1005Metric, symbol Device:C
- added HE74, HE75, HE76, HE77, HE78, HE79, HE80, HE81: MT9102ET, Package_TO_SOT_SMD:SOT-23-3, symbol HE60:MT9102ET
Connections:
- net +3.3VA: now also AM10.16 (VDD), C161.1, C170.1, C172.1, C174.1, C176.1, C178.1, C180.1, C182.1, C184.1, HE74.1 (VCC), HE75.1 (VCC), HE76.1 (VCC), HE77.1 (VCC), HE78.1 (VCC), HE79.1 (VCC), HE80.1 (VCC), HE81.1 (VCC)
- net GND: now also AM10.6 (Inh), C161.2, C170.2, C171.2, C172.2, C173.2, C174.2, C175.2, C176.2, C177.2, C178.2, C179.2, C180.2, C181.2, C182.2, C183.2, C184.2, C185.2, HE74.3 (GND), HE75.3 (GND), HE76.3 (GND), HE77.3 (GND), HE78.3 (GND), HE79.3 (GND), HE80.3 (GND), HE81.3 (GND)
- net MUX_SELECT_0: now also AM10.11 (A)
- net MUX_SELECT_1: now also AM10.10 (B)
- net MUX_SELECT_2: now also AM10.9 (C)
- new net: AM10.7 (VEE), AM10.8 (VSS)
- new net HE70: AM10.13 (X0), C171.1, HE74.2 (OUT)
- new net HE71: AM10.14 (X1), C173.1, HE75.2 (OUT)
- new net HE72: AM10.15 (X2), C175.1, HE76.2 (OUT)
- new net HE73: AM10.12 (X3), C177.1, HE77.2 (OUT)
- new net HE74: AM10.1 (X4), C179.1, HE78.2 (OUT)
- new net HE75: AM10.5 (X5), C181.1, HE79.2 (OUT)
- new net HE76: AM10.2 (X6), C185.1, HE81.2 (OUT)
- new net HE77: AM10.4 (X7), C183.1, HE80.2 (OUT)
- new net MUX_OUT_10: AM10.3 (X)

Commit message: sch: add swd, add uart and adc channel
Parts:
- added J3: JST_SH, Connector_JST:JST_SH_SM04B-SRSS-TB_1x04-1MP_P1.00mm_Horizontal, symbol Connector_Generic_MountingPin:Conn_01x04_MountingPin
- added J4: Conn_01x04_Pin, symbol Connector:Conn_01x04_Pin
- added JP1: SolderJumper_2_Open, symbol Jumper:SolderJumper_2_Open
Connections:
- net +3.3V: now also J4.4 (Pin_4)
- net GND: now also J3.4 (Pin_4), J4.1 (Pin_1)
- net MUX_OUT_10: now also U4.16 (PA2)
- net VBUS: now also JP1.1 (A)
- net UART_TX: now reaches U4.42 (PA9)
- net UART_TX: now also J3.3 (Pin_3)
- net UART_RX: now reaches U4.43 (PA10)
- net UART_RX: now also J3.2 (Pin_2)
- net SWDIO: now reaches U4.46 (PA13)
- net SWDIO: now also J4.3 (Pin_3)
- net SWCLK: now reaches U4.49 (PA14)
- net SWCLK: now also J4.2 (Pin_2)
- new net: J3.1 (Pin_1), JP1.2 (B)
- no-connect marks 41 -> 37

Commit message: layout: add arrows and top 3 block
Parts:
- removed C176: 100n, Capacitor_SMD:C_0402_1005Metric, symbol Device:C
- removed C177: 4.7n, Capacitor_SMD:C_0402_1005Metric, symbol Device:C
- removed HE77: MT9102ET, Package_TO_SOT_SMD:SOT-23-3, symbol HE60:MT9102ET
- added J5: JST_SH, Connector_JST:JST_SH_SM04B-SRSS-TB_1x04-1MP_P1.00mm_Horizontal, symbol Connector_Generic_MountingPin:Conn_01x04_MountingPin
- added JP2: SolderJumper_2_Open, symbol Jumper:SolderJumper_2_Open
Connections:
- net HE73 is gone; now on net HE71: AM10.12 (X3)
- net GND: now also AM10.15 (X2), AM10.7 (VEE), AM10.8 (VSS), J5.4 (Pin_4)
- net HE70: now also AM10.14 (X1); no longer AM10.13 (X0)
- net HE71: no longer AM10.14 (X1)
- net HE72: now also AM10.13 (X0); no longer AM10.15 (X2)
- net HE74: now also AM10.2 (X6); no longer AM10.1 (X4)
- net HE76: now also AM10.1 (X4); no longer AM10.2 (X6)
- net UART_RX: now also J5.2 (Pin_2)
- net UART_TX: now also J5.3 (Pin_3)
- net VBUS: now also JP2.1 (A)
- new net: J5.1 (Pin_1), JP2.2 (B)
- no-connect marks 37 -> 38
Other:
- moved on the sheet: J3, JP1
