File: HE60/HE60.kicad_sch (KiCad schematic)
At the start: 331 parts, among them J1 TYPE-C-31-M-12, J2 JST_SH, SW1 TS-1187A-B-A-B, SW2 TS-1187A-B-A-B, U1 USBLC6-2SC6, U2 TLV75733PDBV, U3 XC6206P332MR-G, U4 AT32F405RCT7, Y1 X322512MSB4SI

Commit message: sch:add extra mux + channels, and JST
Parts:
- removed J2: JST_SH, Connector_JST:JST_SH_SM04B-SRSS-TB_1x04-1MP_P1.00mm_Horizontal, symbol Connector_Generic_MountingPin:Conn_01x04_MountingPin
- added AM10: SN74LV4051A, Package_SO:TSSOP-16_4.4x5mm_P0.65mm, symbol 4xxx:4051
- added C161: 100n, Capacitor_SMD:C_0402_1005Metric, symbol Device:C
- added J3: Conn_01x09_MountingPin, symbol Connector_Generic_MountingPin:Conn_01x09_MountingPin
- added J4: Conn_01x06_MountingPin, symbol Connector_Generic_MountingPin:Conn_01x06_MountingPin
Connections:
- net +3.3VA: now also AM10.16 (VDD), C161.1, J3.1 (Pin_1)
- net GND: now also AM10.4 (X7), AM10.6 (Inh), AM10.7 (VEE), AM10.8 (VSS), C161.2, J3.9 (Pin_9), J4.4 (Pin_4)
- net MUX_SELECT_0: now also AM10.11 (A)
- net MUX_SELECT_1: now also AM10.10 (B)
- net MUX_SELECT_2: now also AM10.9 (C)
- net USB_PLUG_D+: now also J4.3 (Pin_3)
- net USB_PLUG_D-: now also J4.2 (Pin_2)
- net VBUS: now also J4.1 (Pin_1)
- new net AT32_RX: J4.6 (Pin_6)
- new net AT32_TX: J4.5 (Pin_5)
- new net HE70: AM10.15 (X2), J3.2 (Pin_2)
- new net HE71: AM10.12 (X3), J3.3 (Pin_3)
- new net HE72: AM10.1 (X4), J3.4 (Pin_4)
- new net HE73: AM10.5 (X5), J3.5 (Pin_5)
- new net HE74: AM10.2 (X6), J3.6 (Pin_6)
- new net HE75: AM10.13 (X0), J3.7 (Pin_7)
- new net HE76: AM10.14 (X1), J3.8 (Pin_8)
- new net MUX_OUT_10: AM10.3 (X)
- no-connect marks 41 -> 42

Commit message: sch: hookup uart swd mux to mcu, assign foots
Parts:
- added J2: SWD, Connector_PinHeader_2.54mm:PinHeader_1x04_P2.54mm_Vertical, symbol Connector_Generic:Conn_01x04
- J3: footprint (none) -> Connector_JST:JST_SH_SM09B-SRSS-TB_1x09-1MP_P1.00mm_Horizontal
- J4: footprint (none) -> Connector_JST:JST_SH_SM06B-SRSS-TB_1x06-1MP_P1.00mm_Horizontal
Connections:
- net +3.3V: now also J2.1 (Pin_1)
- net AT32_RX: now also U4.43 (PA10)
- net AT32_TX: now also U4.42 (PA9)
- net GND: now also J2.4 (Pin_4)
- net MUX_OUT_10: now also U4.16 (PA2)
- net SWDIO: now reaches U4.46 (PA13)
- net SWDIO: now also J2.2 (Pin_2)
- net SWCLK: now reaches U4.49 (PA14)
- net SWCLK: now also J2.3 (Pin_3)
- no-connect marks 42 -> 37

Commit message: add models for 1u
https://grabcad.com/library/cherry-mx-switches-mx-1
Connections:
- net HE70: now also AM10.12 (X3); no longer AM10.15 (X2)
- net HE71: now also AM10.13 (X0); no longer AM10.12 (X3)
- net HE72: now also AM10.14 (X1); no longer AM10.1 (X4)
- net HE73: now also AM10.15 (X2); no longer AM10.5 (X5)
- net HE74: now also AM10.5 (X5); no longer AM10.2 (X6)
- net HE75: now also AM10.2 (X6); no longer AM10.13 (X0)
- net HE76: now also AM10.1 (X4); no longer AM10.14 (X1)
Changed lines of the file:
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@@
 	(global_label "HE75"
 		(shape input)
-		(at 476.25 208.28 180)
+		(at 476.25 223.52 180)
 		(fields_autoplaced yes)
 		(effects
@@
 		)
 		(property "Intersheetrefs" "${INTERSHEET_REFS}"
-			(at 468.3663 208.28 0)
+			(at 468.3663 223.52 0)
 			(effects
 				(font
@@
 	(global_label "HE74"
 		(shape input)
-		(at 476.25 223.52 180)
+		(at 476.25 220.98 180)
 		(fields_autoplaced yes)
 		(effects
@@
 		)
 		(property "Intersheetrefs" "${INTERSHEET_REFS}"
-			(at 468.3663 223.52 0)
+			(at 468.3663 220.98 0)
 			(effects
 				(font
@@
 	(global_label "HE73"
 		(shape input)
-		(at 476.25 220.98 180)
+		(at 476.25 213.36 180)
 		(fields_autoplaced yes)
 		(effects
@@
 		)
 		(property "Intersheetrefs" "${INTERSHEET_REFS}"
-			(at 468.3663 220.98 0)
+			(at 468.3663 213.36 0)
 			(effects
 				(font
@@
 	(global_label "HE72"
 		(shape input)
-		(at 476.25 218.44 180)
+		(at 476.25 210.82 180)
 		(fields_autoplaced yes)
 		(effects
@@
 		)
 		(property "Intersheetrefs" "${INTERSHEET_REFS}"
-			(at 468.3663 218.44 0)
+			(at 468.3663 210.82 0)
 			(effects
 				(font
@@
 	(global_label "HE76"
 		(shape input)
-		(at 476.25 210.82 180)
+		(at 476.25 218.44 180)
 		(fields_autoplaced yes)
 		(effects
@@
 		)
 		(property "Intersheetrefs" "${INTERSHEET_REFS}"
-			(at 468.3663 210.82 0)
+			(at 468.3663 218.44 0)
 			(effects
 				(font
@@
 	(global_label "HE70"
 		(shape input)
-		(at 476.25 213.36 180)
+		(at 476.25 215.9 180)
 		(fields_autoplaced yes)
 		(effects
@@
 		)
 		(property "Intersheetrefs" "${INTERSHEET_REFS}"
-			(at 468.3663 213.36 0)
+			(at 468.3663 215.9 0)
 			(effects
 				(font
@@
 	(global_label "HE71"
 		(shape input)
-		(at 476.25 215.9 180)
+		(at 476.25 208.28 180)
 		(fields_autoplaced yes)
 		(effects
@@
 		)
 		(property "Intersheetrefs" "${INTERSHEET_REFS}"
-			(at 468.3663 215.9 0)
+			(at 468.3663 208.28 0)
 			(effects
 				(font
