File: hub/hub.kicad_pcb (KiCad board)
At the start: 2 copper layers, 23.9 x 26.1 mm, 15 parts, among them J1 Conn_01x04_Socket, J2 Conn_01x04_Socket, J3 Conn_01x04_Socket, J4 Conn_01x04_Socket, J5 USB_C_Receptacle_USB2.0_14P, U1 CH334F, U5 USBLC6-2SC6, Y2 Crystal_GND24

Commit message: resolve unconnected items
Connections:
- U1 pad 25: (no net) -> GND
Routing:
- net CC2: track 0.00 -> 6.30 mm
- net CC1: track 0.00 -> 6.22 mm
- net GND: track 0.00 -> 4.65 mm, vias 7 -> 69
- net +5V: track 23.5 -> 26.2 mm, vias 4 -> 5
