File: hub/hub.kicad_sch (KiCad schematic)
At the start: 0 parts

Commit message: wip
Parts:
- added F1: Polyfuse_Small, symbol Device:Polyfuse_Small
- added J1, J2, J3, J4: Conn_01x04_Socket, symbol Connector:Conn_01x04_Socket
- added J5: USB_C_Receptacle_USB2.0_14P, symbol Connector:USB_C_Receptacle_USB2.0_14P
- added R1, R2: 5.1K, symbol Device:R
- added U1: CH334F, Package_DFN_QFN:QFN-24-1EP_4x4mm_P0.5mm_EP2.5x2.5mm, symbol symbols:CH334F
- added U5: USBLC6-2SC6, Package_TO_SOT_SMD:SOT-23-6, symbol Power_Protection:USBLC6-2SC6
- added Y1: 12MHz, symbol Device:Crystal
Connections:
- new net: U1.3 (XO), Y1.2
- new net: U1.4 (XI), Y1.1
- new net: J5.A6 (D+), J5.B6 (D+), U5.3 (I/O2)
- new net: J5.A7 (D-), J5.B7 (D-), U5.1 (I/O1)
- new net +5V: F1.1, J5.A4 (VBUS), J5.A9 (VBUS), J5.B4 (VBUS), J5.B9 (VBUS), U1.19 (V5), U5.5 (VBUS)
- new net CC1: J5.A5 (CC1), R2.2
- new net CC2: J5.B5 (CC2), R1.2
- new net DM1: U1.11 (DM1)
- new net DM2: U1.9 (DM2)
- new net DM3: U1.7 (DM3)
- new net DM4: U1.5 (DM4)
- new net DMU: U1.14 (DMU), U5.6 (I/O1)
- new net DP1: U1.12 (DP1)
- new net DP2: U1.10 (DP2)
- new net DP3: U1.8 (DP3)
- new net DP4: U1.6 (DP4)
- new net DPU: U1.15 (DPU), U5.4 (I/O2)
- new net GND: J5.A1 (GND), J5.A12 (GND), J5.B1 (GND), J5.B12 (GND), J5.S1 (SHIELD), R1.1, R2.1, U1.18 (PSELF), U5.2 (GND)
- new net VBUS: F1.2
- no-connect marks 0 -> 10
Other:
- note added: "Is there GND for thsi symbol?"

Commit message: work
Parts:
- removed Y1: 12MHz, symbol Device:Crystal
- added H1, H2, H3, H4: MountingHole, MountingHole:MountingHole_2.2mm_M2_Pad, symbol Mechanical:MountingHole
- added Y2: Crystal_GND24, Crystal:Crystal_SMD_3225-4Pin_3.2x2.5mm, symbol Device:Crystal_GND24
- F1: footprint (none) -> Fuse:Fuse_1812_4532Metric
- J1, J2, J3, J4: footprint (none) -> Connector_JST:JST_SH_SM04B-SRSS-TB_1x04-1MP_P1.00mm_Horizontal
- J5: footprint (none) -> Connector_USB:USB_C_Receptacle_GCT_USB4105-xx-A_16P_TopMnt_Horizontal
- R1, R2: footprint (none) -> Capacitor_SMD:C_0402_1005Metric
Connections:
- net DM1 is gone; now on net D1-: U1.11 (DM1)
- net DM2 is gone; now on net D2-: U1.9 (DM2)
- net DM3 is gone; now on net D3-: U1.7 (DM3)
- net DM4 is gone; now on net D4-: U1.5 (DM4)
- net DP1 is gone; now on net D1+: U1.12 (DP1)
- net DP2 is gone; now on net D2+: U1.10 (DP2)
- net DP3 is gone; now on net D3+: U1.8 (DP3)
- net DP4 is gone; now on net D4+: U1.6 (DP4)
- net GND: now also J1.4 (Pin_4), J2.4 (Pin_4), J3.4 (Pin_4), J4.4 (Pin_4), Y2.2, Y2.4
- net VBUS: now also J1.1 (Pin_1), J2.1 (Pin_1), J3.1 (Pin_1), J4.1 (Pin_1)
- net D1-: now reaches J1.2 (Pin_2)
- net D1+: now reaches J1.3 (Pin_3)
- net D2-: now reaches J2.2 (Pin_2)
- net D2+: now reaches J2.3 (Pin_3)
- net D4-: now reaches J4.2 (Pin_2)
- net D4+: now reaches J4.3 (Pin_3)
- net at U1.3 (XO): now also Y2.1
- net at U1.4 (XI): now also Y2.3
- net D3-: now reaches J3.2 (Pin_2)
- net D3+: now reaches J3.3 (Pin_3)
- net DMU renamed DU_-
- net DPU renamed DU_+
Other:
- moved on the sheet: J1

Commit message: resolve unconnected items
Connections:
- net GND: now also U1.25 (GND)
Changed lines of the file:
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@@
 		(pin "5"
+		)
+		(pin "25"
 		)
 		(instances
@@
 					(unit 1)
 				)
+			)
+		)
+	)
+	(symbol
+		(lib_id "power:GND")
+		(at 231.14 101.6 0)
+		(unit 1)
+		(exclude_from_sim no)
+		(in_bom yes)
+		(on_board yes)
+		(dnp no)
+		(fields_autoplaced yes)
+		(property "Reference" "#PWR019"
+			(at 231.14 107.95 0)
+			(effects
+				(font
+					(size 1.27 1.27)
+				)
+				(hide yes)
+			)
+		)
+		(property "Value" "GND"
+			(at 231.14 106.68 0)
+			(effects
+				(font
+					(size 1.27 1.27)
+				)
+			)
+		)
+		(property "Footprint" ""
+			(at 231.14 101.6 0)
+			(effects
+				(font
+					(size 1.27 1.27)
+				)
+				(hide yes)
+			)
+		)
+		(property "Datasheet" ""
+			(at 231.14 101.6 0)
+			(effects
+				(font
+					(size 1.27 1.27)
+				)
+				(hide yes)
+			)
+		)
+		(property "Description" "Power symbol creates a global label with name \"GND\" , ground"
+			(at 231.14 101.6 0)
+			(effects
+				(font
+					(size 1.27 1.27)
+				)
+				(hide yes)
+			)
+		)
+		(pin "1"
+		)
+		(instances
+			(project ""
+				(path "/625d6237-d56a-462f-8f6f-6bbaf75e0a8d"
+					(reference "#PWR019")
+					(unit 1)
+				)
